File: MINI_TRUNK_6_MAIN/MINI_TRUNK_6_MAIN.kicad_sch (KiCad schematic)
At the start: 7 parts, among them J1 RJ45, J2 RJ45, J3 RJ45, J4 RJ45, J5 RJ45, J6 RJ45, J7 RJ21 Connector

Commit message: nearing completion
Parts:
- added H1, H2, H3, H4: MountingHole, MountingHole:MountingHole_3.2mm_M3, symbol Mechanical:MountingHole
