File: MINI_TRUNK_6_MAIN/MINI_TRUNK_6_MAIN.kicad_pcb (KiCad board)
At the start: 2 copper layers, 102.3 x 34.1 mm, 7 parts, among them J1 RJ45, J2 RJ45, J3 RJ45, J4 RJ45, J5 RJ45, J6 RJ45, J7 RJ21 Connector

Commit message: nearing completion
Parts:
- added H1: MountingHole, MountingHole:MountingHole_3.2mm_M3, F.Cu at (218.4, 69.3)
- added H1: MountingHole, MountingHole:MountingHole_3.2mm_M3, F.Cu at (112.4, 92.7)
- added H2: MountingHole, MountingHole:MountingHole_3.2mm_M3, F.Cu at (112.4, 111.5)
- added H2: MountingHole, MountingHole:MountingHole_3.2mm_M3, F.Cu at (218.4, 50.5)
- added H3: MountingHole, MountingHole:MountingHole_3.2mm_M3, F.Cu at (112.4, 69.3)
- added H3: MountingHole, MountingHole:MountingHole_3.2mm_M3, F.Cu at (218.4, 92.7)
- added H4: MountingHole, MountingHole:MountingHole_3.2mm_M3, F.Cu at (112.4, 50.5)
- added H4: MountingHole, MountingHole:MountingHole_3.2mm_M3, F.Cu at (218.4, 111.5)
- moved J1 2.36 mm to (125.1, 93.6)
- moved J6 2.36 mm to (205.7, 93.6)
- moved J5 1.42 mm to (189.6, 93.6)
- moved J2 1.42 mm to (141.2, 93.6)
- moved J7 0.50 mm to (164.9, 108.8)
- moved J4 0.47 mm to (173.5, 93.6)
- moved J3 0.47 mm to (157.3, 93.6)
Routing:
- net /L3-: track 42.3 -> 35.0 mm
- net /L3+: track 44.0 -> 36.8 mm
- net /L1+: track 37.6 -> 31.5 mm
- net /L2+: track 40.8 -> 34.6 mm
- net /L1-: track 34.6 -> 28.4 mm
- net /L24+: track 36.6 -> 31.3 mm
- net /L2-: track 35.3 -> 30.0 mm
- net /L6+: track 34.1 -> 29.4 mm
- net /L5-: track 27.3 -> 22.9 mm
- net /L7+: track 34.1 -> 30.0 mm
- net /L7-: track 32.0 -> 28.0 mm
- net /L8-: track 32.9 -> 29.0 mm
- net /L8+: track 33.9 -> 30.1 mm
- net /L5+: track 28.7 -> 25.0 mm
- net /L4+: track 40.4 -> 36.7 mm
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Other:
- board size 102.3 x 34.1 mm -> 114.8 x 79.9 mm
- board text added: "HIGH VOLTAGE - DO NOT TOUCH MICRO-TRUNK-6 v0.2"
- board text removed: "1-4"
- board text removed: "13-16"
- board text removed: "17-20"
- board text removed: "21-24"
- board text removed: "5-8"
- board text removed: "9-12"
- board text removed: "HIGH VOLTAGE - DO NOT TOUCH MINI-TRUNK-6 v0.1"

Commit message: Latest changes
Parts:
- removed the H2 at (218.4, 50.5)
- removed the H4 at (112.4, 50.5)
- added H1: MountingHole, MountingHole:MountingHole_3.2mm_M3, F.Cu at (237.5, 92.7)
- added H3: MountingHole, MountingHole:MountingHole_3.2mm_M3, F.Cu at (343.5, 92.7)
- moved H3 132.0 mm to (237.5, 111.5)
- moved H1 132.0 mm to (343.5, 111.5)
Routing:
- net /L13-: track 25.5 -> 32.1 mm
- net /L1+: track 31.5 -> 26.3 mm
- net /L24+: track 31.3 -> 34.1 mm
- net /L23-: track 32.3 -> 33.7 mm
- net /L21-: track 36.1 -> 37.5 mm
- net /L22+: track 37.4 -> 38.5 mm
- net /L9+: track 22.5 -> 23.7 mm
- net /L14-: track 24.6 -> 25.7 mm
- net /L15-: track 21.7 -> 22.8 mm
- net /L22-: track 35.7 -> 36.7 mm
- net /L19-: track 27.8 -> 28.8 mm
- net /L15+: track 24.6 -> 25.5 mm
- net /L19+: track 30.9 -> 31.7 mm
- net /L10+: track 26.5 -> 27.3 mm
- net /L5-: track 22.9 -> 23.8 mm
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Other:
- board size 114.8 x 79.9 mm -> 239.9 x 37.7 mm
- board text added: "01-04"
- board text added: "05-08"
- board text added: "09-12"
- board text added: "13-16"
- board text added: "17-20"
- board text added: "20-24"
