File: MICRO_TRUNK_6_MAIN/MICRO_TRUNK_6_MAIN.kicad_pcb (KiCad board)
At the start: 2 copper layers, 236.3 x 37.7 mm, 15 parts, among them J1 RJ45, J2 RJ45, J3 RJ45, J4 RJ45, J5 RJ45, J6 RJ45, J7 RJ21 Connector

Commit message: Migrate insulators to seperate projects
Parts:
- removed the H1 at (265.2, 99.0)
- removed the H1 at (159.2, 77.9)
- removed the H3 at (159.2, 99.0)
- removed the H3 at (265.2, 77.9)
- moved H3 54.3 mm to (197.6, 83.7)
- moved H4 54.3 mm to (197.6, 105.1)
- moved J3 54.3 mm to (136.6, 87.7)
- moved J5 54.3 mm to (168.8, 87.7)
- moved J7 54.3 mm to (144.1, 102.8)
- moved H1 54.3 mm to (91.6, 83.7)
- moved H2 54.3 mm to (91.6, 105.1)
- moved J2 54.3 mm to (120.5, 87.7)
- moved J4 54.3 mm to (152.7, 87.7)
- moved J6 54.3 mm to (184.9, 87.7)
- moved J1 54.3 mm to (104.4, 87.7)
Other:
- board size 236.3 x 37.7 mm -> 114.8 x 37.7 mm
- board text removed: "01-04"
- board text removed: "05-08"
- board text removed: "09-12"
- board text removed: "13-16"
- board text removed: "17-20"
- board text removed: "20-24"
- board text removed: "B: Ring/-48v A: Tip/0v"
- board text removed: "RJ21 to 6x 4 telephone line 8p8c {dblquote}trunk{dblquote} adapter"
- board text removed: "https://github.com/cu-telecom/MICRO-TRUNK-6"
